Commit message: renaming

File: ros2_ws/src/my_package/urdf/base/my_bot_base.xacro (robot description, xacro)
@@ -72,5 +72,5 @@
             <origin xyz="0 0 -${chassis_height/2}" rpy="-${M_PI/2} 0 0" />
             <geometry>
-                <mesh filename="package://robot_description/meshes/chassis.dae"/>
+                <mesh filename="package://my_package/meshes/chassis.dae"/>
             </geometry>
         </visual>
@@ -101,5 +101,5 @@
             <origin rpy="${M_PI} 0 0" xyz="0 0 0" />
             <geometry>
-                <mesh filename="package://robot_description/meshes/wheels.dae"/>
+                <mesh filename="package://my_package/meshes/wheels.dae"/>
             </geometry>
         </visual>
@@ -130,5 +130,5 @@
             <origin rpy="${M_PI} 0 0" xyz="0 0 0" />
             <geometry>
-                <mesh filename="package://robot_description/meshes/wheels.dae"/>
+                <mesh filename="package://my_package/meshes/wheels.dae"/>
             </geometry>
         </visual>
@@ -159,5 +159,5 @@
             <origin rpy="${M_PI} 0 0" xyz="0 0 0" />
             <geometry>
-                <mesh filename="package://robot_description/meshes/wheels.dae"/>
+                <mesh filename="package://my_package/meshes/wheels.dae"/>
             </geometry>
         </visual>
@@ -188,5 +188,5 @@
             <origin rpy="${M_PI} 0 0" xyz="0 0 0" />
             <geometry>
-                <mesh filename="package://robot_description/meshes/wheels.dae"/>
+                <mesh filename="package://my_package/meshes/wheels.dae"/>
             </geometry>
         </visual>
@@ -206,4 +206,4 @@
         <child link="front_laser" />
     </joint> -->
-    <xacro:include filename="$(find robot_description)/urdf/base/koubot_base.gazebo" />
+    <xacro:include filename="$(find my_package)/urdf/base/koubot_base.gazebo" />
 </robot>
